File: untitled.kicad_sch (KiCad schematic)
At the start: 164 parts

Commit message: day 2 end
Parts:
- renumbered D42 to D?, D8 to D?, D4 to D?, D37 to D?, D59 to D?, D68 to D?, D41 to D?, D17 to D?, D35 to D?, D34 to D?, D3 to D?, D16 to D?, D46 to D?, D67 to D?, D32 to D?, D57 to D?, D75 to D?, D1 to D?, D65 to D?, D61 to D?, D25 to D?, D31 to D?, D18 to D?, D38 to D?, D14 to D?, D54 to D?, D19 to D?, D55 to D?, D69 to D?, D12 to D?, D40 to D?, D30 to D?, D2 to D?, D49 to D?, D48 to D?, D70 to D?, D82 to D?, D44 to D?, D50 to D?, D36 to D?, D80 to D?, D72 to D?, D81 to D?, D43 to D?, D9 to D?, D73 to D?, D63 to D?, D21 to D?, D20 to D?, D6 to D?, D28 to D?, D39 to D?, D10 to D?, D7 to D?, D56 to D?, D27 to D?, D51 to D?, D62 to D?, D77 to D?, D78 to D?, D66 to D?, D26 to D?, D23 to D?, D76 to D?, D74 to D?, D53 to D?, D71 to D?, D64 to D?, D5 to D?, D29 to D?, D52 to D?, D22 to D?, D13 to D?, D79 to D?, D15 to D?, D45 to D?, D47 to D?, D11 to D?, D60 to D?, D58 to D?, D24 to D?, D33 to D?, MX56 to MX?, MX34 to MX?, MX82 to MX?, MX60 to MX?, MX79 to MX?, MX65 to MX?, MX45 to MX?, MX22 to MX?, MX26 to MX?, MX37 to MX?, MX6 to MX?, MX43 to MX?, MX68 to MX?, MX38 to MX?, MX18 to MX?, MX49 to MX?, MX74 to MX?, MX75 to MX?, MX15 to MX?, MX20 to MX?, MX73 to MX?, MX39 to MX?, MX9 to MX?, MX61 to MX?, MX35 to MX?, MX17 to MX?, MX8 to MX?, MX28 to MX?, MX19 to MX?, MX62 to MX?, MX55 to MX?, MX58 to MX?, MX76 to MX?, MX4 to MX?, MX66 to MX?, MX10 to MX?, MX33 to MX?, MX36 to MX?, MX67 to MX?, MX69 to MX?, MX31 to MX?, MX24 to MX?, MX3 to MX?, MX23 to MX?, MX63 to MX?, MX80 to MX?, MX13 to MX?, MX41 to MX?, MX72 to MX?, MX12 to MX?, MX27 to MX?, MX1 to MX?, MX7 to MX?, MX32 to MX?, MX48 to MX?, MX57 to MX?, MX40 to MX?, MX11 to MX?, MX71 to MX?, MX30 to MX?, MX44 to MX?, MX53 to MX?, MX5 to MX?, MX14 to MX?, MX54 to MX?, MX78 to MX?, MX25 to MX?, MX51 to MX?, MX77 to MX?, MX50 to MX?, MX59 to MX?, MX47 to MX?, MX42 to MX?, MX29 to MX?, MX21 to MX?, MX46 to MX?, MX52 to MX?, MX64 to MX?, MX70 to MX?, MX81 to MX?, MX16 to MX?, MX2 to MX?

Commit message: day 3 edit 1
schematic finalized
Parts:
- gave numbers to parts that had none: 164

Commit message: day 3
Parts:
- added D78: D, Diode_SMD:D_SOD-123, symbol Diode:1N4148W
- added MX78: MX_SW_HS, PCM_marbastlib-mx:SW_MX_HS_CPG151101S11_1u, symbol marbastlib-mx:MX_SW_HS_CPG151101S11
- renumbered D2 to D1, D11 to D10, D12 to D11, D13 to D12, D14 to D13, D15 to D14, D1 to D15, D17 to D16, D18 to D17, D19 to D18, D20 to D19, D3 to D2, D21 to D20, D22 to D21, D23 to D22, D24 to D23, D25 to D24, D26 to D25, D27 to D26, D28 to D27, D29 to D28, D30 to D29, D4 to D3, D16 to D30, D32 to D31, D33 to D32, D34 to D33, D35 to D34, D36 to D35, D37 to D36, D38 to D37, D39 to D38, D40 to D39, D5 to D4, D41 to D40, D42 to D41, D43 to D42, D44 to D43, D45 to D44, D31 to D45, D6 to D5, D7 to D6, D8 to D7, D78 to D79, D9 to D8, D79 to D80, D80 to D81, D81 to D82, D82 to D83, D10 to D9, MX78 to MX79, MX79 to MX80, MX80 to MX81, MX81 to MX82, MX82 to MX83
Connections:
- net Col 4: now also MX78.1
- net Row 0: now also D15.1 (K)
- net Row 1: now also D30.1 (K)
- net Row 2: now also D45.1 (K)
- net Row 5: now also D78.2 (A)
- net at MX45.2: now also D45.2 (A)
- net at MX15.2: now also D15.2 (A)
- net at D30.2 (A): now also MX30.2
- new net: D78.1 (K), MX78.2
