File: modular-keyboard-pcb.kicad_pcb (KiCad board)
At the start: 2 copper layers, 320.7 x 126.2 mm, 174 parts, among them J1 Conn_01x02, J2 mag_pogo_01x05, J3 mag_pogo_01x05, J4 mag_pogo_01x05, J5 mag_pogo_01x05, SW1 SW_Push, SW2 SW_Wuerth_450301014042, U1 nice_nano

Commit message: Pcb mostly done
Parts:
- moved D10 119.5 mm to (183.0, 38.3)
- moved D14 119.5 mm to (259.2, 38.3)
- moved D15 119.5 mm to (302.1, 38.3)
- moved D28 119.5 mm to (230.7, 62.1)
- moved D29 119.5 mm to (259.2, 62.1)
- moved D30 119.5 mm to (302.1, 62.1)
- moved D40 119.5 mm to (183.0, 81.2)
- moved D45 119.5 mm to (302.1, 81.2)
- moved D56 119.5 mm to (206.9, 100.2)
- moved D59 119.5 mm to (302.1, 100.2)
- moved D67 119.5 mm to (159.2, 119.3)
- moved D71 119.5 mm to (242.6, 119.3)
- moved D73 119.5 mm to (302.1, 119.3)
- moved D80 119.5 mm to (230.7, 138.3)
- moved D83 119.5 mm to (295.0, 143.1)
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
Commit message: PCB done?
Routing:
- net Row 0: track 388.7 -> 387.9 mm
- net Col 9: track 486.6 -> 487.4 mm
- net Row 1: track 347.1 -> 346.6 mm
- added copper zone on B.Cu, net GND
- added copper zone on F.Cu, net GND
Changed lines of the file:
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@@
 	)
 	(segment
-		(start 248.6025 143.8275)
-		(end -7.77875 143.8275)
+		(start 281.14625 85.09)
+		(end 268.2875 72.23125)
 		(width 0.254)
 		(layer "F.Cu")
@@
 	)
 	(segment
-		(start -7.77875 143.8275)
-		(end -10.5705 141.03575)
+		(start 268.2875 72.23125)
+		(end 268.2875 56.1975)
 		(width 0.254)
 		(layer "F.Cu")
@@
 	)
 	(segment
-		(start 281.14625 85.09)
-		(end 268.2875 72.23125)
+		(start 281.14625 145.415)
+		(end 281.14625 85.09)
 		(width 0.254)
 		(layer "F.Cu")
@@
 	)
 	(segment
-		(start 251.7775 147.0025)
-		(end 248.6025 143.8275)
+		(start 279.55875 147.0025)
+		(end 281.14625 145.415)
 		(width 0.254)
 		(layer "F.Cu")
 		(net "Col 9")
 	)
-	(segment
-		(start 268.2875 72.23125)
-		(end 268.2875 56.1975)
-		(width 0.254)
-		(layer "F.Cu")
+	(via
+		(at 279.55875 147.0025)
+		(size 0.8)
+		(drill 0.3)
+		(layers "F.Cu" "B.Cu")
 		(net "Col 9")
 	)
 	(segment
-		(start 279.55875 147.0025)
-		(end 251.7775 147.0025)
+		(start 248.888603 143.66875)
+		(end 252.222353 147.0025)
 		(width 0.254)
-		(layer "F.Cu")
+		(layer "B.Cu")
 		(net "Col 9")
 	)
 	(segment
-		(start 281.14625 145.415)
-		(end 281.14625 85.09)
+		(start 296.70375 147.0025)
+		(end 304.5755 139.13075)
 		(width 0.254)
-		(layer "F.Cu")
+		(layer "B.Cu")
 		(net "Col 9")
 	)
 	(segment
-		(start -10.5705 106.9045)
-		(end -11.7475 105.7275)
+		(start 252.222353 147.0025)
+		(end 279.55875 147.0025)
 		(width 0.254)
-		(layer "F.Cu")
+		(layer "B.Cu")
 		(net "Col 9")
 	)
 	(segment
-		(start 279.55875 147.0025)
-		(end 281.14625 145.415)
+		(start -11.7475 105.7275)
+		(end -9.82025 107.65475)
 		(width 0.254)
-		(layer "F.Cu")
+		(layer "B.Cu")
 		(net "Col 9")
 	)
 	(segment
-		(start -10.5705 141.03575)
-		(end -10.5705 106.9045)
+		(start -9.82025 141.786)
+		(end -7.9375 143.66875)
 		(width 0.254)
-		(layer "F.Cu")
+		(layer "B.Cu")
 		(net "Col 9")
 	)
-	(via
-		(at 279.55875 147.0025)
-		(size 0.8)
-		(drill 0.3)
-		(layers "F.Cu" "B.Cu")
+	(segment
+		(start 304.5755 139.13075)
+		(end 304.5755 106.9045)
+		(width 0.254)
+		(layer "B.Cu")
 		(net "Col 9")
 	)
 	(segment
-		(start 279.55875 147.0025)
-		(end 295.43375 147.0025)
+		(start 304.5755 106.9045)
+		(end 305.7525 105.7275)
 		(width 0.254)
 		(layer "B.Cu")
@@
 	)
 	(segment
-		(start 295.43375 147.0025)
-		(end 304.5755 137.86075)
+		(start 279.55875 147.0025)
+		(end 296.70375 147.0025)
 		(width 0.254)
 		(layer "B.Cu")
@@
 	)
 	(segment
-		(start 304.5755 137.86075)
-		(end 304.5755 106.9045)
+		(start -9.82025 107.65475)
+		(end -9.82025 141.786)
 		(width 0.254)
 		(layer "B.Cu")
@@
 	)
 	(segment
-		(start 304.5755 106.9045)
-		(end 305.7525 105.7275)
+		(start -7.9375 143.66875)
+		(end 248.888603 143.66875)
 		(width 0.254)
 		(layer "B.Cu")
@@
 	)
 	(segment
-		(start 279.6335 24.3635)
-		(end 266.4665 24.3635)
+		(start 264.4775 44.60875)
+		(end 264.4775 26.3525)
 		(width 0.508)
 		(layer "F.Cu")
@@
 	)
 	(segment
-		(start 264.4775 26.3525)
-		(end 264.4775 44.60875)
+		(start 266.8985 23.9315)
+		(end 279.2015 23.9315)
 		(width 0.508)
 		(layer "F.Cu")
@@
 	)
 	(segment
-		(start 264.4775 44.60875)
-		(end 262.89 46.19625)
+		(start 264.4775 26.3525)
+		(end 266.8985 23.9315)
 		(width 0.508)
 		(layer "F.Cu")
@@
 	)
 	(segment
-		(start 266.4665 24.3635)
-		(end 264.4775 26.3525)
+		(start 283.5275 28.2575)
+		(end 283.05125 28.2575)
 		(width 0.508)
 		(layer "F.Cu")
@@
 	)
 	(segment
-		(start 262.89 46.19625)
-		(end 247.9675 46.19625)
+		(start 247.9675 46.19625)
+		(end 262.89 46.19625)
 		(width 0.508)
 		(layer "F.Cu")
@@
 	)
 	(segment
-		(start 283.5275 28.2575)
-		(end 279.6335 24.3635)
+		(start 262.89 46.19625)
+		(end 264.4775 44.60875)
 		(width 0.508)
 		(layer "F.Cu")
@@
 	)
 	(segment
-		(start 283.5275 28.2575)
-		(end 283.05125 28.2575)
+		(start 279.2015 23.9315)
+		(end 283.5275 28.2575)
 		(width 0.508)
 		(layer "F.Cu")
@@
 	)
 	(segment
-		(start -10.95375 57.30875)
-		(end -9.36625 58.89625)
-		(width 0.254)
-		(layer "B.Cu")
-		(net "Row 0")
-	)
-	(segment
 		(start 221.13875 39.94)
 		(end 240.18875 39.94)
@@
 	)
 	(segment
+		(start -10.31875 63.65875)
+		(end -10.31875 57.94375)
+		(width 0.254)
+		(layer "B.Cu")
+		(net "Row 0")
+	)
+	(segment
+		(start -11.7475 65.0875)
+		(end -10.31875 63.65875)
+		(width 0.254)
+		(layer "B.Cu")
+		(net "Row 0")
+	)
+	(segment
 		(start 263.68375 43.02125)
 		(end 263.68375 54.13375)
@@
 	)
 	(segment
-		(start -3.90375 39.94)
-		(end -10.95375 46.99)
-		(width 0.254)
-		(layer "B.Cu")
-		(net "Row 0")
-	)
-	(segment
 		(start 144.93875 39.94)
 		(end 163.98875 39.94)
@@
 	)
 	(segment
-		(start -10.95375 46.99)
-		(end -10.95375 57.30875)
+		(start -10.95375 57.30875)
+		(end -10.95375 46.99)
 		(width 0.254)
 		(layer "B.Cu")
@@
 	)
 	(segment
-		(start 183.03875 39.94)
-		(end 202.08875 39.94)
+		(start -3.90375 39.94)
+		(end 2.06375 39.94)
 		(width 0.254)
 		(layer "B.Cu")
@@
 	)
 	(segment
-		(start -9.36625 58.89625)
-		(end -9.36625 62.70625)
+		(start 183.03875 39.94)
+		(end 202.08875 39.94)
 		(width 0.254)
 		(layer "B.Cu")
@@
 	)
 	(segment
-		(start 2.06375 39.94)
+		(start -10.95375 46.99)
 		(end -3.90375 39.94)
 		(width 0.254)
@@
 	)
 	(segment
-		(start 260.6025 39.94)
-		(end 263.68375 43.02125)
+		(start -10.31875 57.94375)
+		(end -10.95375 57.30875)
 		(width 0.254)
 		(layer "B.Cu")
@@
 	)
 	(segment
-		(start -9.36625 62.70625)
-		(end -11.7475 65.0875)
+		(start 260.6025 39.94)
+		(end 263.68375 43.02125)
 		(width 0.254)
 		(layer "B.Cu")
@@
 	)
 	(segment
+		(start 304.165 67.6275)
+		(end 305.7525 67.6275)
+		(width 0.254)
+		(layer "B.Cu")
+		(net "Row 1")
+	)
+	(segment
 		(start 230.66375 63.7525)
 		(end 259.23875 63.7525)
@@
 	)
 	(segment
-		(start 2.06375 63.7525)
-		(end -7.8725 63.7525)
+		(start 302.10125 65.56375)
+		(end 304.165 67.6275)
 		(width 0.254)
 		(layer "B.Cu")
@@
 	)
 	(segment
-		(start 78.26375 63.7525)
-		(end 97.31375 63.7525)
+		(start 2.06375 63.7525)
+		(end -7.8725 63.7525)
 		(width 0.254)
 		(layer "B.Cu")
@@
 	)
 	(segment
-		(start 304.165 67.6275)
-		(end 305.7525 67.6275)
+		(start 78.26375 63.7525)
+		(end 97.31375 63.7525)
 		(width 0.254)
 		(layer "B.Cu")
@@
 	)
 	(segment
-		(start 302.10125 63.7525)
-		(end 302.10125 63.97625)
-		(width 0.254)
-		(layer "B.Cu")
-		(net "Row 1")
-	)
-	(segment
-		(start 303.37125 64.4525)
-		(end 303.37125 66.83375)
-		(width 0.254)
-		(layer "B.Cu")
-		(net "Row 1")
-	)
-	(segment
 		(start 278.311 50.619)
 		(end 282.8925 46.0375)
@@
 	)
 	(segment
-		(start 302.10125 63.7525)
-		(end 302.67125 63.7525)
-		(width 0.254)
-		(layer "B.Cu")
-		(net "Row 1")
-	)
-	(segment
 		(start 173.51375 63.7525)
 		(end 192.56375 63.7525)
@@
 	)
 	(segment
-		(start 302.67125 63.7525)
-		(end 303.37125 64.4525)
-		(width 0.254)
-		(layer "B.Cu")
-		(net "Row 1")
-	)
-	(segment
 		(start 283.5275 46.0375)
 		(end 284.95625 46.0375)
@@
 	)
 	(segment
-		(start 303.37125 66.83375)
-		(end 304.165 67.6275)
+		(start 302.10125 63.7525)
+		(end 302.10125 65.56375)
 		(width 0.254)
 		(layer "B.Cu")
@@
 		(net "Net-(D61-A)")
 	)
+	(zone
+		(net "GND")
+		(layers "F.Cu" "B.Cu")
+		(hatch edge 0.5)
+		(connect_pads
+			(clearance 0.5)
+		)
+		(min_thickness 0.25)
+		(fill yes
+			(thermal_gap 0.5)
+			(thermal_bridge_width 0.5)
+			(island_removal_mode 2)
+			(island_area_min 9.999999)
+		)
+		(polygon
+			(pts
+				(xy -14.2875 148.43125) (xy 309.5625 150.8125) (xy 311.15 17.4625) (xy -16.66875 19.05)
+			)
+		)
+	)
 	(embedded_fonts no)

Commit message: final pcb?
Parts:
- moved SW2 19.9 mm to (246.9, 66.1)
Routing:
- net Col 9: track 487.4 -> 589.1 mm
- net Col 6: track 216.7 -> 200.8 mm
- net Bat+: track 57.7 -> 64.6 mm
- net Col 0: track 516.3 -> 514.8 mm, vias 0 -> 1

Commit message: pcb final tweak before review
Routing:
- net Col 8: track 408.6 -> 407.3 mm
Changed lines of the file:
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@@
 	)
 	(segment
-		(start 304.165 58.89625)
-		(end 304.95875 58.1025)
-		(width 0.254)
-		(layer "F.Cu")
-		(net "Col 8")
-	)
-	(segment
-		(start 306.54625 57.30875)
-		(end 306.54625 53.34)
+		(start 306 57.5)
+		(end 306 54)
 		(width 0.254)
 		(layer "F.Cu")
@@
 	)
 	(segment
-		(start 294.16375 40.9575)
-		(end 283.5275 40.9575)
-		(width 0.254)
-		(layer "F.Cu")
-		(net "Col 8")
-	)
-	(segment
-		(start 305.7525 58.1025)
-		(end 306.54625 57.30875)
+		(start 305.030625 58.030625)
+		(end 305.469375 58.030625)
 		(width 0.254)
 		(layer "F.Cu")
@@
 	)
 	(segment
-		(start 306.54625 53.34)
-		(end 294.16375 40.9575)
+		(start 292.9575 40.9575)
+		(end 283.5275 40.9575)
+		(width 0.254)
+		(layer "F.Cu")
+		(net "Col 8")
+	)
+	(segment
+		(start 304.165 60.96)
+		(end 304.165 58.89625)
+		(width 0.254)
+		(layer "F.Cu")
+		(net "Col 8")
+	)
+	(segment
+		(start 304.165 58.89625)
+		(end 305.030625 58.030625)
 		(width 0.254)
 		(layer "F.Cu")
@@
 	)
 	(segment
-		(start 304.165 60.96)
-		(end 304.165 58.89625)
+		(start 305.469375 58.030625)
+		(end 306 57.5)
+		(width 0.254)
+		(layer "F.Cu")
+		(net "Col 8")
+	)
+	(segment
+		(start 306 54)
+		(end 292.9575 40.9575)
 		(width 0.254)
 		(layer "F.Cu")
@@
 		(width 0.254)
 		(layer "F.Cu")
-		(net "Col 8")
-	)
-	(segment
-		(start 304.95875 58.1025)
-		(end 305.7525 58.1025)
-		(width 0.254)
-		(layer "F.Cu")
